Commit message: feat: update hand URDF joint limits, mimic ratios, and thumb zero
- Thumb abduction: shift metacarpal joint origin by +3 deg; limits 0~90 deg
- Thumb MCP/PIP limits: 0~62 deg / 0~66 deg; PIP mimic 1.0945x
- Four-finger PIP limits: 0~97 deg; mimic 1.131 / 1.267 / 1.252 / 1.271
- Keep thumb MCP/PIP origin compensation (+9 deg / +6 deg)
- Sync .urdf and .urdf.xacro; bump version to 1.1.0

File: urdf/revo2_left_hand.urdf (robot description, URDF)
Before this commit: robot brainco_revo2_lefthand_urdf, 22 links, 21 joints
Joints:
- joint left_index_distal_joint: limit lower=0 upper=1.63 effort=2 velocity=2.2685 -> lower=0 upper=1.69297 effort=2 velocity=2.2685; mimic joint=left_index_proximal_joint multiplier=1.155 offset=0 -> joint=left_index_proximal_joint multiplier=1.131 offset=0
- joint left_middle_distal_joint: limit lower=0 upper=1.63 effort=2 velocity=2.2685 -> lower=0 upper=1.69297 effort=2 velocity=2.2685; mimic joint=left_middle_proximal_joint multiplier=1.155 offset=0 -> joint=left_middle_proximal_joint multiplier=1.267 offset=0
- joint left_pinky_distal_joint: limit lower=0 upper=1.63 effort=2 velocity=2.2685 -> lower=0 upper=1.69297 effort=2 velocity=2.2685; mimic joint=left_pinky_proximal_joint multiplier=1.155 offset=0 -> joint=left_pinky_proximal_joint multiplier=1.271 offset=0
- joint left_ring_distal_joint: limit lower=0 upper=1.63 effort=2 velocity=2.2685 -> lower=0 upper=1.69297 effort=2 velocity=2.2685; mimic joint=left_ring_proximal_joint multiplier=1.155 offset=0 -> joint=left_ring_proximal_joint multiplier=1.252 offset=0
- joint left_thumb_distal_joint: limit lower=0 upper=1.03 effort=1.1 velocity=2.5303 -> lower=0 upper=1.15192 effort=1.1 velocity=2.5303; mimic joint=left_thumb_proximal_joint multiplier=1 offset=0 -> joint=left_thumb_proximal_joint multiplier=1.0945 offset=0; origin xyz=0 -0.052 0 rpy=0 0 0 -> xyz=0 -0.052 0 rpy=0.10472 0 0
- joint left_thumb_metacarpal_joint: origin xyz=0.0045 -0.019 0.027825 rpy=0 0 0.16787 -> xyz=0.0045 -0.019 0.027825 rpy=0 0 0.22023
- joint left_thumb_proximal_joint: limit lower=0 upper=1.03 effort=1.1 velocity=2.5303 -> lower=0 upper=1.08210 effort=1.1 velocity=2.5303; origin xyz=0 -0.014227 0 rpy=-0.17488 0.23736 -0.16787 -> xyz=0 -0.014227 0 rpy=-0.33153 0.23736 -0.16787

File: urdf/revo2_left_hand.urdf.xacro (robot description, xacro)
@@ -56,5 +56,6 @@
   </link>
   <joint name="left_thumb_metacarpal_joint" type="revolute">
-    <origin xyz="0.0045 -0.019 0.027825" rpy="0 0 0.16787" />
+    <!-- 零位重定义：新 q=0 对应旧坐标 +3deg（Stark2.0 URDF 2026-08-14） -->
+    <origin xyz="0.0045 -0.019 0.027825" rpy="0 0 0.22023" />
     <parent link="left_base_link" />
     <child link="left_thumb_metacarpal_link" />
@@ -99,5 +100,5 @@
     <child link="left_thumb_proximal_link" />
     <axis xyz="-1 0 0" />
-    <limit lower="0" upper="1.03" effort="1.1" velocity="2.5303" />
+    <limit lower="0" upper="1.08210" effort="1.1" velocity="2.5303" />
   </joint>
   <link name="left_thumb_distal_link">
@@ -129,6 +130,6 @@
     <child link="left_thumb_distal_link" />
     <axis xyz="-1 0 0" />
-    <limit lower="0" upper="1.03" effort="1.1" velocity="2.5303" />
-    <mimic joint="left_thumb_proximal_joint" multiplier="0.691851" offset="0.0395854" />
+    <limit lower="0" upper="1.15192" effort="1.1" velocity="2.5303" />
+    <mimic joint="left_thumb_proximal_joint" multiplier="1.0945" offset="0" />
   </joint>
   <link name="left_thumb_tip_link">
@@ -224,6 +225,6 @@
     <child link="left_index_distal_link" />
     <axis xyz="0 1 0" />
-    <limit lower="0" upper="1.63" effort="2" velocity="2.2685" />
-    <mimic joint="left_index_proximal_joint" multiplier="1.155" offset="0" />
+    <limit lower="0" upper="1.69297" effort="2" velocity="2.2685" />
+    <mimic joint="left_index_proximal_joint" multiplier="1.131" offset="0" />
   </joint>
   <link name="left_index_tip_link">
@@ -319,6 +320,6 @@
     <child link="left_middle_distal_link" />
     <axis xyz="0 1 0" />
-    <limit lower="0" upper="1.63" effort="2" velocity="2.2685" />
-    <mimic joint="left_middle_proximal_joint" multiplier="1.155" offset="0" />
+    <limit lower="0" upper="1.69297" effort="2" velocity="2.2685" />
+    <mimic joint="left_middle_proximal_joint" multiplier="1.267" offset="0" />
   </joint>
   <link name="left_middle_tip_link">
@@ -414,6 +415,6 @@
     <child link="left_ring_distal_link" />
     <axis xyz="0 1 0" />
-    <limit lower="0" upper="1.63" effort="2" velocity="2.2685" />
-    <mimic joint="left_ring_proximal_joint" multiplier="1.155" offset="0" />
+    <limit lower="0" upper="1.69297" effort="2" velocity="2.2685" />
+    <mimic joint="left_ring_proximal_joint" multiplier="1.252" offset="0" />
   </joint>
   <link name="left_ring_tip_link">
@@ -509,6 +510,6 @@
     <child link="left_pinky_distal_link" />
     <axis xyz="0 1 0" />
-    <limit lower="0" upper="1.63" effort="2" velocity="2.2685" />
-    <mimic joint="left_pinky_proximal_joint" multiplier="1.155" offset="0" />
+    <limit lower="0" upper="1.69297" effort="2" velocity="2.2685" />
+    <mimic joint="left_pinky_proximal_joint" multiplier="1.271" offset="0" />
   </joint>
   <link name="left_pinky_tip_link">

File: urdf/revo2_right_hand.urdf (robot description, URDF)
Before this commit: robot brainco_revo2_righthand_urdf, 22 links, 21 joints
Joints:
- joint right_index_distal_joint: limit lower=0 upper=1.63 effort=2 velocity=2.2685 -> lower=0 upper=1.69297 effort=2 velocity=2.2685; mimic joint=right_index_proximal_joint multiplier=1.155 offset=0 -> joint=right_index_proximal_joint multiplier=1.131 offset=0
- joint right_middle_distal_joint: limit lower=0 upper=1.63 effort=2 velocity=2.2685 -> lower=0 upper=1.69297 effort=2 velocity=2.2685; mimic joint=right_middle_proximal_joint multiplier=1.155 offset=0 -> joint=right_middle_proximal_joint multiplier=1.267 offset=0
- joint right_pinky_distal_joint: limit lower=0 upper=1.63 effort=2 velocity=2.2685 -> lower=0 upper=1.69297 effort=2 velocity=2.2685; mimic joint=right_pinky_proximal_joint multiplier=1.155 offset=0 -> joint=right_pinky_proximal_joint multiplier=1.271 offset=0
- joint right_ring_distal_joint: limit lower=0 upper=1.63 effort=2 velocity=2.2685 -> lower=0 upper=1.69297 effort=2 velocity=2.2685; mimic joint=right_ring_proximal_joint multiplier=1.155 offset=0 -> joint=right_ring_proximal_joint multiplier=1.252 offset=0
- joint right_thumb_distal_joint: limit lower=0 upper=1.03 effort=1.1 velocity=2.5303 -> lower=0 upper=1.15192 effort=1.1 velocity=2.5303; mimic joint=right_thumb_proximal_joint multiplier=1 offset=0 -> joint=right_thumb_proximal_joint multiplier=1.0945 offset=0; origin xyz=0 0.052 0 rpy=0 0 0 -> xyz=0 0.052 0 rpy=-0.10472 0 0
- joint right_thumb_metacarpal_joint: origin xyz=0.005619 0.019867 0.027825 rpy=0 0 -0.16787 -> xyz=0.005619 0.019867 0.027825 rpy=0 0 -0.22023
- joint right_thumb_proximal_joint: limit lower=0 upper=1.03 effort=1.1 velocity=2.5303 -> lower=0 upper=1.08210 effort=1.1 velocity=2.5303; origin xyz=0 0.014227 0 rpy=0.17488 0.23736 0.16787 -> xyz=0 0.014227 0 rpy=0.33153 0.23736 0.16787

File: urdf/revo2_right_hand.urdf.xacro (robot description, xacro)
@@ -56,5 +56,6 @@
     </link>
     <joint name="right_thumb_metacarpal_joint" type="revolute">
-      <origin xyz="0.005619 0.019867 0.027825" rpy="0 0 -0.16787" />
+      <!-- 零位重定义：新 q=0 对应旧坐标 +3deg（Stark2.0 URDF 2026-08-14） -->
+      <origin xyz="0.005619 0.019867 0.027825" rpy="0 0 -0.22023" />
       <parent link="right_base_link" />
       <child link="right_thumb_metacarpal_link" />
@@ -90,5 +91,5 @@
       <child link="right_thumb_proximal_link" />
       <axis xyz="1 0 0" />
-      <limit lower="0" upper="1.03" effort="1.1" velocity="2.5303" />
+      <limit lower="0" upper="1.08210" effort="1.1" velocity="2.5303" />
     </joint>
     <link name="right_thumb_distal_link">
@@ -120,6 +121,6 @@
       <child link="right_thumb_distal_link" />
       <axis xyz="1 0 0" />
-      <limit lower="0" upper="1.03" effort="1.1" velocity="2.5303" />
-      <mimic joint="right_thumb_proximal_joint" multiplier="0.691851" offset="0.0395854" />
+      <limit lower="0" upper="1.15192" effort="1.1" velocity="2.5303" />
+      <mimic joint="right_thumb_proximal_joint" multiplier="1.0945" offset="0" />
     </joint>
     <link name="right_thumb_tip_link" />
@@ -214,6 +215,6 @@
       <child link="right_index_distal_link" />
       <axis xyz="0 1 0" />
-      <limit lower="0" upper="1.63" effort="2" velocity="2.2685" />
-      <mimic joint="right_index_proximal_joint" multiplier="1.155" offset="0" />
+      <limit lower="0" upper="1.69297" effort="2" velocity="2.2685" />
+      <mimic joint="right_index_proximal_joint" multiplier="1.131" offset="0" />
     </joint>
     <link name="right_index_tip_link" />
@@ -308,6 +309,6 @@
       <child link="right_middle_distal_link" />
       <axis xyz="0 1 0" />
-      <limit lower="0" upper="1.63" effort="2" velocity="2.2685" />
-      <mimic joint="right_middle_proximal_joint" multiplier="1.155" offset="0" />
+      <limit lower="0" upper="1.69297" effort="2" velocity="2.2685" />
+      <mimic joint="right_middle_proximal_joint" multiplier="1.267" offset="0" />
     </joint>
     <link name="right_middle_tip_link" />
@@ -402,6 +403,6 @@
       <child link="right_ring_distal_link" />
       <axis xyz="0 1 0" />
-      <limit lower="0" upper="1.63" effort="2" velocity="2.2685" />
-      <mimic joint="right_ring_proximal_joint" multiplier="1.155" offset="0" />
+      <limit lower="0" upper="1.69297" effort="2" velocity="2.2685" />
+      <mimic joint="right_ring_proximal_joint" multiplier="1.252" offset="0" />
     </joint>
     <link name="right_ring_tip_link" />
@@ -496,6 +497,6 @@
       <child link="right_pinky_distal_link" />
       <axis xyz="0 1 0" />
-      <limit lower="0" upper="1.63" effort="2" velocity="2.2685" />
-      <mimic joint="right_pinky_proximal_joint" multiplier="1.155" offset="0" />
+      <limit lower="0" upper="1.69297" effort="2" velocity="2.2685" />
+      <mimic joint="right_pinky_proximal_joint" multiplier="1.271" offset="0" />
     </joint>
     <link name="right_pinky_tip_link" />

Commit message: fix: align thumb abduction and MCP limits with mass-production version (20260818)
- Thumb abduction: 0~89 deg (upper 1.55334 rad)
- Thumb MCP: 0~60 deg (upper 1.04720 rad)
- Sync .urdf and .urdf.xacro; bump version to 1.1.1

File: urdf/revo2_left_hand.urdf (robot description, URDF)
Before this commit: robot brainco_revo2_lefthand_urdf, 22 links, 21 joints
Joints:
- joint left_thumb_metacarpal_joint: limit lower=0 upper=1.57 effort=0.5 velocity=2.6175 -> lower=0 upper=1.55334 effort=0.5 velocity=2.6175
- joint left_thumb_proximal_joint: limit lower=0 upper=1.08210 effort=1.1 velocity=2.5303 -> lower=0 upper=1.04720 effort=1.1 velocity=2.5303

File: urdf/revo2_left_hand.urdf.xacro (robot description, xacro)
@@ -61,5 +61,5 @@
     <child link="left_thumb_metacarpal_link" />
     <axis xyz="0 0 1" />
-    <limit lower="0" upper="1.57" effort="0.5" velocity="2.6175" />
+    <limit lower="0" upper="1.55334" effort="0.5" velocity="2.6175" />
   </joint>
   <link name="left_thumb_proximal_link">
@@ -100,5 +100,5 @@
     <child link="left_thumb_proximal_link" />
     <axis xyz="-1 0 0" />
-    <limit lower="0" upper="1.08210" effort="1.1" velocity="2.5303" />
+    <limit lower="0" upper="1.04720" effort="1.1" velocity="2.5303" />
   </joint>
   <link name="left_thumb_distal_link">

File: urdf/revo2_right_hand.urdf (robot description, URDF)
Before this commit: robot brainco_revo2_righthand_urdf, 22 links, 21 joints
Joints:
- joint right_thumb_metacarpal_joint: limit lower=0 upper=1.57 effort=0.5 velocity=2.6175 -> lower=0 upper=1.55334 effort=0.5 velocity=2.6175
- joint right_thumb_proximal_joint: limit lower=0 upper=1.08210 effort=1.1 velocity=2.5303 -> lower=0 upper=1.04720 effort=1.1 velocity=2.5303

File: urdf/revo2_right_hand.urdf.xacro (robot description, xacro)
@@ -61,5 +61,5 @@
       <child link="right_thumb_metacarpal_link" />
       <axis xyz="0 0 -1" />
-      <limit lower="0" upper="1.57" effort="0.5" velocity="2.6175" />
+      <limit lower="0" upper="1.55334" effort="0.5" velocity="2.6175" />
     </joint>
     <link name="right_thumb_proximal_link">
@@ -91,5 +91,5 @@
       <child link="right_thumb_proximal_link" />
       <axis xyz="1 0 0" />
-      <limit lower="0" upper="1.08210" effort="1.1" velocity="2.5303" />
+      <limit lower="0" upper="1.04720" effort="1.1" velocity="2.5303" />
     </joint>
     <link name="right_thumb_distal_link">
